Commit message: sep 19 add panda_trajectory_following_mujoco.py planner concretize xddot: tweak

File: examples/planar_urdf_2_joints.urdf (robot description, URDF)
Before this commit: robot panda_description, 5 links, 4 joints
Links:
- removed link panda_link0
- removed link panda_link1
- removed link panda_link2
- removed link panda_link4
- added link link0, mass 1.00; collision sphere radius=0.1; visual sphere radius=0.1
- added link link1, mass 1.0; collision cylinder length=1.0 radius=0.1; visual cylinder length=1.0 radius=0.1
- added link link2, mass 1.0; collision cylinder length=1.0 radius=0.1; visual cylinder length=1.0 radius=0.1
- added link link4, mass 0.0001; collision sphere radius=0.1; visual sphere radius=0.1
Joints:
- removed joint panda_joint1
- removed joint panda_joint2
- removed joint panda_joint4
- added joint joint1: type revolute, parent link0, child link1, origin xyz=0 0 0.0 rpy=0 0 0, axis 1 0 0, limit lower=-2.8973 upper=2.8973 effort=87 velocity=2.1750
- added joint joint2: type revolute, parent link1, child link2, origin xyz=0 0 1.1 rpy=0 0 0, axis 1 0 0, limit lower=-2.8973 upper=2.8973 effort=87 velocity=2.1750
- added joint joint4: type fixed, parent link2, child link4, origin xyz=0 0 1.2 rpy=0 0 0, axis 1 0 0
- joint robot_to_world: child panda_link0 -> link0

Commit message: planar robot fix

File: examples/planar_urdf_2_joints.urdf (robot description, URDF)
Before this commit: robot description, 5 links, 4 joints
Links:
- removed link link4
- added link link3, mass 0.0001; collision sphere radius=0.1; visual sphere radius=0.1
Joints:
- removed joint joint4
- added joint joint3: type fixed, parent link2, child link3, origin xyz=0 0 1.2 rpy=0 0 0, axis 1 0 0
